File: hardware/mie1001_daq_simple/mie1001_daq_simple.kicad_pcb (KiCad board)
At the start: 2 copper layers, 68.6 x 53.3 mm, 34 parts, among them J1 SIGNAL IN, J2 QPS OUT, J3 TRIG IN, J4 SPARE ADC A1-A3, J5 DET IN (SMA), U1 ADS1115 breakout, U2 MCP4725 breakout, U3 LMP7721, U4 MCP6002

Commit message: Shield rev E, Digi-Key ordering, shield firmware, self-test data, enclosure
- Simple shield rev E: fixes from an embedded-systems design review (guard ring
  closed under the LMP7721 and free of solder mask, 100k/100k VREF divider, A4/A5
  wired to SDA/SCL, JP1 mass-command read-back on ADS A2, flood-fill guard check
  that fails on rev D). Parts re-verified at Digi-Key; fab/digikey_bom.csv added,
  README covers ordering the bare PCB via DigiKey PCB Builder and hand-soldering.
- firmware/DAQ_shield_scan: preamp current (A1-A3), zero, settled mass scan with
  50 Hz window averaging, A2 command read-back, trigger on D8, self-check.
- Team sketches: ioannis_DAC_3V (now corrects for the real 5 V rail) and the
  SparkFun MCP4725 waveform example (credited, licence kept).
- data/2026-09-20_selftest: first real ADS1115/MCP4725 self-test results + plots.
- hardware/enclosure: first transparent PETG enclosure idea (OpenSCAD, STL, renders).

Co-Authored-By: Claude Opus 5.5 <noreply@anthropic.com>
Parts:
- added JP1: QPS readback, Jumper:SolderJumper-2_P1.3mm_Bridged_RoundedPad1.0x1.5mm, F.Cu at (127.4, 86.0)
- R8, R9: value 10k -> 100k
Connections:
- ARD1 pad 13: (no net) -> /SDA
- ARD1 pad 14: (no net) -> /SCL
Routing:
- net /SCL: track 71.3 -> 121.6 mm, vias 8 -> 6
- net /SDA: track 57.9 -> 89.9 mm, vias 6 -> 8
- net /AIN2: track 13.8 -> 24.0 mm, vias 2 -> 5
- net /QPS: track 25.6 -> 31.6 mm
- net /TRIG_EXT: track 22.1 -> 26.9 mm, vias 2 -> 4
- net +5V: track 113.3 -> 111.3 mm, vias 17 -> 15
- net /TIA_OUT: track 9.87 -> 11.6 mm, vias 0 -> 2
- net /DET_IN: track 4.97 -> 6.26 mm
- net /PRE_OUT: track 37.6 -> 36.9 mm
- net /VREF: track 74.4 -> 73.7 mm, vias 8 -> 6
- net /TRIG: track 68.1 -> 68.0 mm, vias 8 -> 3
Other:
- board text added: "A2=QPS"
- board text added: "MIE1001 Team 5 simple DAQ rev E"
- board text added: "simple DAQ shield rev E"
- board text removed: "MIE1001 Team 5 simple DAQ rev D"
- board text removed: "simple DAQ shield rev D"

Commit message: Shield rev E: neutral silkscreen text (possum kept), Digi-Key ordering files
Co-Authored-By: Claude Opus 5.5 <noreply@anthropic.com>
Other:
- board text added: "DATA ACQUISITION"
- board text added: "IMAGING ENGINEERING 2026"
- board text added: "MIE1001 TEAM 5"
- board text removed: "MIE1001 SUFFERING"
- board text removed: "MIGHTY MACHINE GODS"
- board text removed: "WE PRAY TO THE"
