File: hardware/mie1001_daq_simple/mie1001_daq_simple.kicad_sch (KiCad schematic)
At the start: 31 parts, among them J1 SIGNAL IN, J2 QPS OUT, J3 TRIG IN, J4 SPARE ADC A1-A3, J5 DET IN (SMA), U1 ADS1115 breakout, U2 MCP4725 breakout, U3 LMP7721, U4 MCP6002

Commit message: Shield rev E, Digi-Key ordering, shield firmware, self-test data, enclosure
- Simple shield rev E: fixes from an embedded-systems design review (guard ring
  closed under the LMP7721 and free of solder mask, 100k/100k VREF divider, A4/A5
  wired to SDA/SCL, JP1 mass-command read-back on ADS A2, flood-fill guard check
  that fails on rev D). Parts re-verified at Digi-Key; fab/digikey_bom.csv added,
  README covers ordering the bare PCB via DigiKey PCB Builder and hand-soldering.
- firmware/DAQ_shield_scan: preamp current (A1-A3), zero, settled mass scan with
  50 Hz window averaging, A2 command read-back, trigger on D8, self-check.
- Team sketches: ioannis_DAC_3V (now corrects for the real 5 V rail) and the
  SparkFun MCP4725 waveform example (credited, licence kept).
- data/2026-09-20_selftest: first real ADS1115/MCP4725 self-test results + plots.
- hardware/enclosure: first transparent PETG enclosure idea (OpenSCAD, STL, renders).

Co-Authored-By: Claude Opus 5.5 <noreply@anthropic.com>
Parts:
- added JP1: QPS readback, Jumper:SolderJumper-2_P1.3mm_Bridged_RoundedPad1.0x1.5mm, symbol DAQ:SolderJumper_2_Bridged
- C1: Manufacturer Vishay -> Vishay Beyschlag/Draloric/BC Components
- C2: Digi-Key P/N 490-1403-1-ND -> 1276-1027-1-ND; MPN GRM1885C1H100JA01D -> CL10C100JB8NNNC; Manufacturer Murata -> Samsung Electro-Mechanics; Note MUST be fitted: without it the preamp oscillates with the c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 -> C0G/NP0 only. MUST be fitted: without it the preamp oscilla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
- C3, C7: Digi-Key P/N 1276-1000-1-ND -> 732-8013-1-ND; MPN CL10B104KB8NNNC -> 885012206095; Manufacturer Samsung -> Wurth Elektronik
- C4: Digi-Key P/N 1276-2891-1-ND -> 587-4334-1-ND; MPN CL21A106KAYNNNE -> TMK212BBJ106KGHT; Manufacturer Samsung -> Taiyo Yuden
- C5: Digi-Key P/N 1276-1860-1-ND -> 1276-1102-1-ND; LCSC C15849 -> C5673; MPN CL10A105KB8NNNC -> CL10A105KA8NNNC; Manufacturer Samsung -> Samsung Electro-Mechanics; Note (none) -> VREF output capacitor (25 V is plenty at 2.5 V).; Rating 1uF X5R 50V 0603 -> 1uF X5R 25V 0603
- C6: Digi-Key P/N 1276-1860-1-ND -> 1276-1102-1-ND; LCSC C15849 -> C5673; MPN CL10A105KB8NNNC -> CL10A105KA8NNNC; Manufacturer Samsung -> Samsung Electro-Mechanics; Rating 1uF X5R 50V 0603 -> 1uF X5R 25V 0603
- J4: Manufacturer Sullins -> Sullins Connector Solutions
- R1, R10, R11, R2, R3, R5, R7: Manufacturer Yageo -> YAGEO
- R4: Digi-Key P/N 10KQBK-ND -> 13-CFR-25JB-52-10K-ND; Manufacturer Yageo -> YAGEO
- R6: Manufacturer Stackpole -> Stackpole Electronics Inc; Note 100 MOhm feedback: 1 nA -> 0.1 V. Guard the pads, keep them clean, no flux residue. JLC/LCSC has no Stackpole HVCB stock: use Uniroyal 1206W4F1006T5E (C59781), 1% +-100 ppm/C. -> 100 MOhm feedback: 1 nA -> 0.1 V. Guard the pads, keep them clean, no flux residue. Must stay a high-value low-leakage 1 % part: do not substitute a general-purpose 1206. (The LCSC column is only for the optional JLC route: Uniroyal 1206W4F1006T5E.)
- R8: value 10k -> 100k; Digi-Key P/N 311-10.0KHRCT-ND -> 311-100KHRCT-ND; LCSC C25804 -> C25803; MPN RC0603FR-0710KL -> RC0603FR-07100KL; Manufacturer Yageo -> YAGEO; Note (none) -> Rev E: 100k/100k (was 10k/10k). With C4 10 uF the divider n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; Rating 10k 1% 0603 -> 100k 1% 0603
- R9: value 10k -> 100k; Digi-Key P/N 311-10.0KHRCT-ND -> 311-100KHRCT-ND; LCSC C25804 -> C25803; MPN RC0603FR-0710KL -> RC0603FR-07100KL; Manufacturer Yageo -> YAGEO; Rating 10k 1% 0603 -> 100k 1% 0603
- U2: MPN BOB-12918 -> 12918; Manufacturer SparkFun -> SparkFun Electronics; Note The footprint is a 1x6 female header (PPTC061LFBN-RC). Pull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 -> SparkFun BOB-12918. The footprint is a 1x6 female header (P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
- U3: Note Electrometer preamp (3 fA typical input bias). Guard ring (VREF) on both layers around pins 1/8 and the feedback parts, no solder mask there. Clean flux off after soldering. -> Electrometer preamp (3 fA typical input bias). Guard ring (VREF) on both layers around pins 1/8 and the feedback parts, closed under the chip between pins 2 and 7; the guard copper is left free of solder mask (rev E), tracks and the gaps next to them stay masked. Clean flux off after soldering.
- U4: Manufacturer Microchip -> Microchip Technology
Connections:
- net AIN2: now also JP1.1 (A)
- net QPS: now also JP1.2 (B)
- net SCL: now also ARD1.14 (SCL/A5)
- net SDA: now also ARD1.13 (SDA/A4)
- no-connect marks 24 -> 22
Other:
- note added: "J4 (ADS1115 inputs, not the UNO's): 1 = A1 preamp out, 2 = A2 (QPS read-back while JP1 is bridged), 3 = A3 VREF 2.5 V, 4 = GND. Pins 1-3 are for a meter or scope only."
- note added: "QPS OUT: mass command 0-5 V to the Extrel controller (Team 4) JP1 (bridged by default) reads it back on ADS1115 A2. Cut JP1's copper bridge to free A2 / J4-2."
- note added: "Reads U1 and sets U2 over I2C, sends the data to the laptop over USB. This board plugs on top of it. Pin NAMES shown (D2, D8, SDA...), as printed on the UNO. SDA/A4 and SCL/A5 are the SAME signals as SDA and SCL: the shield connects both (for clones without SDA/SCL pins). Never use A4/A5 as analog inputs. Your board: Uno R3 CH340G clone, IOREF is labelled 5V."
- note removed: "J4 (ADS1115 inputs, not the UNO's): 1 = A1 preamp out, 2 = A2 spare, 3 = A3 VREF 2.5 V, 4 = GND. Pins 1 and 3 are for a meter or scope only."
- note removed: "QPS OUT: mass command 0-5 V to the Extrel controller (Team 4)"
- note removed: "Reads U1 and sets U2 over I2C, sends the data to the laptop over USB. This board plugs on top of it. Pin NAMES shown (D2, D8, SDA...), as printed on the UNO. SDA/A4 and SCL/A5 are the SAME wires as SDA and SCL inside the UNO: keep A4 and A5 free. Your board: Uno R3 CH340G clone, IOREF is labelled 5V."
